Commit message: new parameters

File: assets/urdf/bdx/urdf/bdx.urdf (robot description, URDF)
Before this commit: robot bdx, 20 links, 19 joints
Joints:
- joint head_pitch: limit lower=-0.69813170079773179122 upper=0.69813170079773179122 effort=0.58 velocity=20 -> lower=-0.69813170079773179122 upper=0.69813170079773179122 effort=0.58 velocity=10.7
- joint head_yaw: limit lower=-2.0943951023931952626 upper=2.0943951023931952626 effort=0.58 velocity=20 -> lower=-2.0943951023931952626 upper=2.0943951023931952626 effort=0.58 velocity=10.7
- joint left_ankle: limit lower=-1.570796326794896558 upper=1.570796326794896558 effort=0.58 velocity=20 -> lower=-1.570796326794896558 upper=1.570796326794896558 effort=0.58 velocity=10.7
- joint left_antenna: limit lower=-1.1344640137963142301 upper=2.0943951023931952626 effort=0.58 velocity=20 -> lower=-1.1344640137963142301 upper=2.0943951023931952626 effort=0.58 velocity=10.7
- joint left_hip_pitch: limit lower=-0.52359877559829881566 upper=1.570796326794896558 effort=0.58 velocity=20 -> lower=-0.52359877559829881566 upper=1.570796326794896558 effort=0.58 velocity=10.7
- joint left_hip_roll: limit lower=-1.570796326794896558 upper=0.43633231299858238339 effort=0.58 velocity=20 -> lower=-1.570796326794896558 upper=0.43633231299858238339 effort=0.58 velocity=10.7
- joint left_hip_yaw: limit lower=-0.69813170079773179122 upper=0.69813170079773179122 effort=0.58 velocity=20 -> lower=-0.69813170079773179122 upper=0.69813170079773179122 effort=0.58 velocity=10.7
- joint left_knee: limit lower=-2.0943951023931952626 upper=2.0943951023931952626 effort=0.58 velocity=20 -> lower=-2.0943951023931952626 upper=2.0943951023931952626 effort=0.58 velocity=10.7
- joint neck_pitch: limit lower=-1.3089969389957472057 upper=0.1745329251994329478 effort=0.58 velocity=20 -> lower=-1.3089969389957472057 upper=0.1745329251994329478 effort=0.58 velocity=10.7
- joint right_ankle: limit lower=-1.570796326794896558 upper=1.570796326794896558 effort=0.58 velocity=20 -> lower=-1.570796326794896558 upper=1.570796326794896558 effort=0.58 velocity=10.7
- joint right_antenna: limit lower=-2.0943951023931952626 upper=1.1344640137963142301 effort=0.58 velocity=20 -> lower=-2.0943951023931952626 upper=1.1344640137963142301 effort=0.58 velocity=10.7
- joint right_hip_pitch: limit lower=-0.52359877559829881566 upper=1.570796326794896558 effort=0.58 velocity=20 -> lower=-0.52359877559829881566 upper=1.570796326794896558 effort=0.58 velocity=10.7
- joint right_hip_roll: limit lower=-1.570796326794896558 upper=0.43633231299858238339 effort=0.58 velocity=20 -> lower=-1.570796326794896558 upper=0.43633231299858238339 effort=0.58 velocity=10.7
- joint right_hip_yaw: limit lower=-0.69813170079773179122 upper=0.69813170079773179122 effort=0.58 velocity=20 -> lower=-0.69813170079773179122 upper=0.69813170079773179122 effort=0.58 velocity=10.7
- joint right_knee: limit lower=-2.0943951023931952626 upper=2.0943951023931952626 effort=0.58 velocity=20 -> lower=-2.0943951023931952626 upper=2.0943951023931952626 effort=0.58 velocity=10.7

Commit message: higher standing pose

File: assets/urdf/bdx/urdf/bdx.urdf (robot description, URDF)
Before this commit: robot bdx, 20 links, 19 joints
Joints:
- joint head_pitch: limit lower=-0.69813170079773179122 upper=0.69813170079773179122 effort=0.58 velocity=10.7 -> lower=-0.69813170079773179122 upper=0.69813170079773179122 effort=0.52 velocity=10.7
- joint head_yaw: limit lower=-2.0943951023931952626 upper=2.0943951023931952626 effort=0.58 velocity=10.7 -> lower=-2.0943951023931952626 upper=2.0943951023931952626 effort=0.52 velocity=10.7
- joint left_ankle: limit lower=-1.570796326794896558 upper=1.570796326794896558 effort=0.58 velocity=10.7 -> lower=-1.570796326794896558 upper=1.570796326794896558 effort=0.52 velocity=10.7
- joint left_antenna: limit lower=-1.1344640137963142301 upper=2.0943951023931952626 effort=0.58 velocity=10.7 -> lower=-1.1344640137963142301 upper=2.0943951023931952626 effort=0.52 velocity=10.7
- joint left_hip_pitch: limit lower=-0.52359877559829881566 upper=1.570796326794896558 effort=0.58 velocity=10.7 -> lower=-0.52359877559829881566 upper=1.570796326794896558 effort=0.52 velocity=10.7
- joint left_hip_roll: limit lower=-1.570796326794896558 upper=0.43633231299858238339 effort=0.58 velocity=10.7 -> lower=-1.570796326794896558 upper=0.43633231299858238339 effort=0.52 velocity=10.7
- joint left_hip_yaw: limit lower=-0.69813170079773179122 upper=0.69813170079773179122 effort=0.58 velocity=10.7 -> lower=-0.69813170079773179122 upper=0.69813170079773179122 effort=0.52 velocity=10.7
- joint left_knee: limit lower=-2.0943951023931952626 upper=2.0943951023931952626 effort=0.58 velocity=10.7 -> lower=-2.0943951023931952626 upper=2.0943951023931952626 effort=0.52 velocity=10.7
- joint neck_pitch: limit lower=-1.3089969389957472057 upper=0.1745329251994329478 effort=0.58 velocity=10.7 -> lower=-1.3089969389957472057 upper=0.1745329251994329478 effort=0.52 velocity=10.7
- joint right_ankle: limit lower=-1.570796326794896558 upper=1.570796326794896558 effort=0.58 velocity=10.7 -> lower=-1.570796326794896558 upper=1.570796326794896558 effort=0.52 velocity=10.7
- joint right_antenna: limit lower=-2.0943951023931952626 upper=1.1344640137963142301 effort=0.58 velocity=10.7 -> lower=-2.0943951023931952626 upper=1.1344640137963142301 effort=0.52 velocity=10.7
- joint right_hip_pitch: limit lower=-0.52359877559829881566 upper=1.570796326794896558 effort=0.58 velocity=10.7 -> lower=-0.52359877559829881566 upper=1.570796326794896558 effort=0.52 velocity=10.7
- joint right_hip_roll: limit lower=-1.570796326794896558 upper=0.43633231299858238339 effort=0.58 velocity=10.7 -> lower=-1.570796326794896558 upper=0.43633231299858238339 effort=0.52 velocity=10.7
- joint right_hip_yaw: limit lower=-0.69813170079773179122 upper=0.69813170079773179122 effort=0.58 velocity=10.7 -> lower=-0.69813170079773179122 upper=0.69813170079773179122 effort=0.52 velocity=10.7
- joint right_knee: limit lower=-2.0943951023931952626 upper=2.0943951023931952626 effort=0.58 velocity=10.7 -> lower=-2.0943951023931952626 upper=2.0943951023931952626 effort=0.52 velocity=10.7

Commit message: 6V

File: assets/urdf/bdx/urdf/bdx.urdf (robot description, URDF)
Before this commit: robot bdx, 20 links, 19 joints
Joints:
- joint head_pitch: limit lower=-0.69813170079773179122 upper=0.69813170079773179122 effort=0.52 velocity=10.7 -> lower=-0.69813170079773179122 upper=0.69813170079773179122 effort=0.6 velocity=10.7
- joint head_yaw: limit lower=-2.0943951023931952626 upper=2.0943951023931952626 effort=0.52 velocity=10.7 -> lower=-2.0943951023931952626 upper=2.0943951023931952626 effort=0.6 velocity=10.7
- joint left_ankle: limit lower=-1.570796326794896558 upper=1.570796326794896558 effort=0.52 velocity=10.7 -> lower=-1.570796326794896558 upper=1.570796326794896558 effort=0.6 velocity=10.7
- joint left_antenna: limit lower=-1.1344640137963142301 upper=2.0943951023931952626 effort=0.52 velocity=10.7 -> lower=-1.1344640137963142301 upper=2.0943951023931952626 effort=0.6 velocity=10.7
- joint left_hip_pitch: limit lower=-0.52359877559829881566 upper=1.570796326794896558 effort=0.52 velocity=10.7 -> lower=-0.52359877559829881566 upper=1.570796326794896558 effort=0.6 velocity=10.7
- joint left_hip_roll: limit lower=-1.570796326794896558 upper=0.43633231299858238339 effort=0.52 velocity=10.7 -> lower=-1.570796326794896558 upper=0.43633231299858238339 effort=0.6 velocity=10.7
- joint left_hip_yaw: limit lower=-0.69813170079773179122 upper=0.69813170079773179122 effort=0.52 velocity=10.7 -> lower=-0.69813170079773179122 upper=0.69813170079773179122 effort=0.6 velocity=10.7
- joint left_knee: limit lower=-2.0943951023931952626 upper=2.0943951023931952626 effort=0.52 velocity=10.7 -> lower=-2.0943951023931952626 upper=2.0943951023931952626 effort=0.6 velocity=10.7
- joint neck_pitch: limit lower=-1.3089969389957472057 upper=0.1745329251994329478 effort=0.52 velocity=10.7 -> lower=-1.3089969389957472057 upper=0.1745329251994329478 effort=0.6 velocity=10.7
- joint right_ankle: limit lower=-1.570796326794896558 upper=1.570796326794896558 effort=0.52 velocity=10.7 -> lower=-1.570796326794896558 upper=1.570796326794896558 effort=0.6 velocity=10.7
- joint right_antenna: limit lower=-2.0943951023931952626 upper=1.1344640137963142301 effort=0.52 velocity=10.7 -> lower=-2.0943951023931952626 upper=1.1344640137963142301 effort=0.6 velocity=10.7
- joint right_hip_pitch: limit lower=-0.52359877559829881566 upper=1.570796326794896558 effort=0.52 velocity=10.7 -> lower=-0.52359877559829881566 upper=1.570796326794896558 effort=0.6 velocity=10.7
- joint right_hip_roll: limit lower=-1.570796326794896558 upper=0.43633231299858238339 effort=0.52 velocity=10.7 -> lower=-1.570796326794896558 upper=0.43633231299858238339 effort=0.6 velocity=10.7
- joint right_hip_yaw: limit lower=-0.69813170079773179122 upper=0.69813170079773179122 effort=0.52 velocity=10.7 -> lower=-0.69813170079773179122 upper=0.69813170079773179122 effort=0.6 velocity=10.7
- joint right_knee: limit lower=-2.0943951023931952626 upper=2.0943951023931952626 effort=0.52 velocity=10.7 -> lower=-2.0943951023931952626 upper=2.0943951023931952626 effort=0.6 velocity=10.7

Commit message: xc

File: assets/urdf/bdx/urdf/bdx.urdf (robot description, URDF)
Before this commit: robot bdx, 20 links, 19 joints
Joints:
- joint head_pitch: limit lower=-0.69813170079773179122 upper=0.69813170079773179122 effort=0.6 velocity=10.7 -> lower=-0.69813170079773179122 upper=0.69813170079773179122 effort=0.9 velocity=10.7
- joint head_yaw: limit lower=-2.0943951023931952626 upper=2.0943951023931952626 effort=0.6 velocity=10.7 -> lower=-2.0943951023931952626 upper=2.0943951023931952626 effort=0.9 velocity=10.7
- joint left_ankle: limit lower=-1.570796326794896558 upper=1.570796326794896558 effort=0.6 velocity=10.7 -> lower=-1.570796326794896558 upper=1.570796326794896558 effort=0.9 velocity=10.7
- joint left_antenna: limit lower=-1.1344640137963142301 upper=2.0943951023931952626 effort=0.6 velocity=10.7 -> lower=-1.1344640137963142301 upper=2.0943951023931952626 effort=0.9 velocity=10.7
- joint left_hip_pitch: limit lower=-0.52359877559829881566 upper=1.570796326794896558 effort=0.6 velocity=10.7 -> lower=-0.52359877559829881566 upper=1.570796326794896558 effort=0.9 velocity=10.7
- joint left_hip_roll: limit lower=-1.570796326794896558 upper=0.43633231299858238339 effort=0.6 velocity=10.7 -> lower=-1.570796326794896558 upper=0.43633231299858238339 effort=0.9 velocity=10.7
- joint left_hip_yaw: limit lower=-0.69813170079773179122 upper=0.69813170079773179122 effort=0.6 velocity=10.7 -> lower=-0.69813170079773179122 upper=0.69813170079773179122 effort=0.9 velocity=10.7
- joint left_knee: limit lower=-2.0943951023931952626 upper=2.0943951023931952626 effort=0.6 velocity=10.7 -> lower=-2.0943951023931952626 upper=2.0943951023931952626 effort=0.9 velocity=10.7
- joint neck_pitch: limit lower=-1.3089969389957472057 upper=0.1745329251994329478 effort=0.6 velocity=10.7 -> lower=-1.3089969389957472057 upper=0.1745329251994329478 effort=0.9 velocity=10.7
- joint right_ankle: limit lower=-1.570796326794896558 upper=1.570796326794896558 effort=0.6 velocity=10.7 -> lower=-1.570796326794896558 upper=1.570796326794896558 effort=0.9 velocity=10.7
- joint right_antenna: limit lower=-2.0943951023931952626 upper=1.1344640137963142301 effort=0.6 velocity=10.7 -> lower=-2.0943951023931952626 upper=1.1344640137963142301 effort=0.9 velocity=10.7
- joint right_hip_pitch: limit lower=-0.52359877559829881566 upper=1.570796326794896558 effort=0.6 velocity=10.7 -> lower=-0.52359877559829881566 upper=1.570796326794896558 effort=0.9 velocity=10.7
- joint right_hip_roll: limit lower=-1.570796326794896558 upper=0.43633231299858238339 effort=0.6 velocity=10.7 -> lower=-1.570796326794896558 upper=0.43633231299858238339 effort=0.9 velocity=10.7
- joint right_hip_yaw: limit lower=-0.69813170079773179122 upper=0.69813170079773179122 effort=0.6 velocity=10.7 -> lower=-0.69813170079773179122 upper=0.69813170079773179122 effort=0.9 velocity=10.7
- joint right_knee: limit lower=-2.0943951023931952626 upper=2.0943951023931952626 effort=0.6 velocity=10.7 -> lower=-2.0943951023931952626 upper=2.0943951023931952626 effort=0.9 velocity=10.7

Commit message: xc knees

File: assets/urdf/bdx/urdf/bdx.urdf (robot description, URDF)
Before this commit: robot bdx, 20 links, 19 joints
Joints:
- joint head_pitch: limit lower=-0.69813170079773179122 upper=0.69813170079773179122 effort=0.9 velocity=10.7 -> lower=-0.69813170079773179122 upper=0.69813170079773179122 effort=0.6 velocity=10.7
- joint head_yaw: limit lower=-2.0943951023931952626 upper=2.0943951023931952626 effort=0.9 velocity=10.7 -> lower=-2.0943951023931952626 upper=2.0943951023931952626 effort=0.6 velocity=10.7
- joint left_ankle: limit lower=-1.570796326794896558 upper=1.570796326794896558 effort=0.9 velocity=10.7 -> lower=-1.570796326794896558 upper=1.570796326794896558 effort=0.6 velocity=10.7
- joint left_antenna: limit lower=-1.1344640137963142301 upper=2.0943951023931952626 effort=0.9 velocity=10.7 -> lower=-1.1344640137963142301 upper=2.0943951023931952626 effort=0.6 velocity=10.7
- joint left_hip_pitch: limit lower=-0.52359877559829881566 upper=1.570796326794896558 effort=0.9 velocity=10.7 -> lower=-0.52359877559829881566 upper=1.570796326794896558 effort=0.6 velocity=10.7
- joint left_hip_roll: limit lower=-1.570796326794896558 upper=0.43633231299858238339 effort=0.9 velocity=10.7 -> lower=-1.570796326794896558 upper=0.43633231299858238339 effort=0.6 velocity=10.7
- joint left_hip_yaw: limit lower=-0.69813170079773179122 upper=0.69813170079773179122 effort=0.9 velocity=10.7 -> lower=-0.69813170079773179122 upper=0.69813170079773179122 effort=0.6 velocity=10.7
- joint neck_pitch: limit lower=-1.3089969389957472057 upper=0.1745329251994329478 effort=0.9 velocity=10.7 -> lower=-1.3089969389957472057 upper=0.1745329251994329478 effort=0.6 velocity=10.7
- joint right_ankle: limit lower=-1.570796326794896558 upper=1.570796326794896558 effort=0.9 velocity=10.7 -> lower=-1.570796326794896558 upper=1.570796326794896558 effort=0.6 velocity=10.7
- joint right_antenna: limit lower=-2.0943951023931952626 upper=1.1344640137963142301 effort=0.9 velocity=10.7 -> lower=-2.0943951023931952626 upper=1.1344640137963142301 effort=0.6 velocity=10.7
- joint right_hip_pitch: limit lower=-0.52359877559829881566 upper=1.570796326794896558 effort=0.9 velocity=10.7 -> lower=-0.52359877559829881566 upper=1.570796326794896558 effort=0.6 velocity=10.7
- joint right_hip_roll: limit lower=-1.570796326794896558 upper=0.43633231299858238339 effort=0.9 velocity=10.7 -> lower=-1.570796326794896558 upper=0.43633231299858238339 effort=0.6 velocity=10.7
- joint right_hip_yaw: limit lower=-0.69813170079773179122 upper=0.69813170079773179122 effort=0.9 velocity=10.7 -> lower=-0.69813170079773179122 upper=0.69813170079773179122 effort=0.6 velocity=10.7

Commit message: effort 1.0

File: assets/urdf/bdx/urdf/bdx.urdf (robot description, URDF)
Before this commit: robot bdx, 20 links, 19 joints
Joints:
- joint head_pitch: limit lower=-0.69813170079773179122 upper=0.69813170079773179122 effort=0.6 velocity=10.7 -> lower=-0.69813170079773179122 upper=0.69813170079773179122 effort=1.0 velocity=10.7
- joint head_yaw: limit lower=-2.0943951023931952626 upper=2.0943951023931952626 effort=0.6 velocity=10.7 -> lower=-2.0943951023931952626 upper=2.0943951023931952626 effort=1.0 velocity=10.7
- joint left_ankle: limit lower=-1.570796326794896558 upper=1.570796326794896558 effort=0.6 velocity=10.7 -> lower=-1.570796326794896558 upper=1.570796326794896558 effort=1.0 velocity=10.7
- joint left_antenna: limit lower=-1.1344640137963142301 upper=2.0943951023931952626 effort=0.6 velocity=10.7 -> lower=-1.1344640137963142301 upper=2.0943951023931952626 effort=1.0 velocity=10.7
- joint left_hip_pitch: limit lower=-0.52359877559829881566 upper=1.570796326794896558 effort=0.6 velocity=10.7 -> lower=-0.52359877559829881566 upper=1.570796326794896558 effort=1.0 velocity=10.7
- joint left_hip_roll: limit lower=-1.570796326794896558 upper=0.43633231299858238339 effort=0.6 velocity=10.7 -> lower=-1.570796326794896558 upper=0.43633231299858238339 effort=1.0 velocity=10.7
- joint left_hip_yaw: limit lower=-0.69813170079773179122 upper=0.69813170079773179122 effort=0.6 velocity=10.7 -> lower=-0.69813170079773179122 upper=0.69813170079773179122 effort=1.0 velocity=10.7
- joint left_knee: limit lower=-2.0943951023931952626 upper=2.0943951023931952626 effort=0.9 velocity=10.7 -> lower=-2.0943951023931952626 upper=2.0943951023931952626 effort=1.0 velocity=10.7
- joint neck_pitch: limit lower=-1.3089969389957472057 upper=0.1745329251994329478 effort=0.6 velocity=10.7 -> lower=-1.3089969389957472057 upper=0.1745329251994329478 effort=1.0 velocity=10.7
- joint right_ankle: limit lower=-1.570796326794896558 upper=1.570796326794896558 effort=0.6 velocity=10.7 -> lower=-1.570796326794896558 upper=1.570796326794896558 effort=1.0 velocity=10.7
- joint right_antenna: limit lower=-2.0943951023931952626 upper=1.1344640137963142301 effort=0.6 velocity=10.7 -> lower=-2.0943951023931952626 upper=1.1344640137963142301 effort=1.0 velocity=10.7
- joint right_hip_pitch: limit lower=-0.52359877559829881566 upper=1.570796326794896558 effort=0.6 velocity=10.7 -> lower=-0.52359877559829881566 upper=1.570796326794896558 effort=1.0 velocity=10.7
- joint right_hip_roll: limit lower=-1.570796326794896558 upper=0.43633231299858238339 effort=0.6 velocity=10.7 -> lower=-1.570796326794896558 upper=0.43633231299858238339 effort=1.0 velocity=10.7
- joint right_hip_yaw: limit lower=-0.69813170079773179122 upper=0.69813170079773179122 effort=0.6 velocity=10.7 -> lower=-0.69813170079773179122 upper=0.69813170079773179122 effort=1.0 velocity=10.7
- joint right_knee: limit lower=-2.0943951023931952626 upper=2.0943951023931952626 effort=0.9 velocity=10.7 -> lower=-2.0943951023931952626 upper=2.0943951023931952626 effort=1.0 velocity=10.7

Commit message: try

File: assets/urdf/bdx/urdf/bdx.urdf (robot description, URDF)
Before this commit: robot bdx, 20 links, 19 joints
Joints:
- joint head_pitch: limit lower=-0.69813170079773179122 upper=0.69813170079773179122 effort=1.0 velocity=10.7 -> lower=-0.69813170079773179122 upper=0.69813170079773179122 effort=0.52 velocity=10.7
- joint head_yaw: limit lower=-2.0943951023931952626 upper=2.0943951023931952626 effort=1.0 velocity=10.7 -> lower=-2.0943951023931952626 upper=2.0943951023931952626 effort=0.52 velocity=10.7
- joint left_ankle: limit lower=-1.570796326794896558 upper=1.570796326794896558 effort=1.0 velocity=10.7 -> lower=-1.570796326794896558 upper=1.570796326794896558 effort=0.52 velocity=10.7
- joint left_antenna: limit lower=-1.1344640137963142301 upper=2.0943951023931952626 effort=1.0 velocity=10.7 -> lower=-1.1344640137963142301 upper=2.0943951023931952626 effort=0.52 velocity=10.7
- joint left_hip_pitch: limit lower=-0.52359877559829881566 upper=1.570796326794896558 effort=1.0 velocity=10.7 -> lower=-0.52359877559829881566 upper=1.570796326794896558 effort=0.52 velocity=10.7
- joint left_hip_roll: limit lower=-1.570796326794896558 upper=0.43633231299858238339 effort=1.0 velocity=10.7 -> lower=-1.570796326794896558 upper=0.43633231299858238339 effort=0.52 velocity=10.7
- joint left_hip_yaw: limit lower=-0.69813170079773179122 upper=0.69813170079773179122 effort=1.0 velocity=10.7 -> lower=-0.69813170079773179122 upper=0.69813170079773179122 effort=0.52 velocity=10.7
- joint left_knee: limit lower=-2.0943951023931952626 upper=2.0943951023931952626 effort=1.0 velocity=10.7 -> lower=-2.0943951023931952626 upper=2.0943951023931952626 effort=0.52 velocity=10.7
- joint neck_pitch: limit lower=-1.3089969389957472057 upper=0.1745329251994329478 effort=1.0 velocity=10.7 -> lower=-1.3089969389957472057 upper=0.1745329251994329478 effort=0.52 velocity=10.7
- joint right_ankle: limit lower=-1.570796326794896558 upper=1.570796326794896558 effort=1.0 velocity=10.7 -> lower=-1.570796326794896558 upper=1.570796326794896558 effort=0.52 velocity=10.7
- joint right_antenna: limit lower=-2.0943951023931952626 upper=1.1344640137963142301 effort=1.0 velocity=10.7 -> lower=-2.0943951023931952626 upper=1.1344640137963142301 effort=0.52 velocity=10.7
- joint right_hip_pitch: limit lower=-0.52359877559829881566 upper=1.570796326794896558 effort=1.0 velocity=10.7 -> lower=-0.52359877559829881566 upper=1.570796326794896558 effort=0.52 velocity=10.7
- joint right_hip_roll: limit lower=-1.570796326794896558 upper=0.43633231299858238339 effort=1.0 velocity=10.7 -> lower=-1.570796326794896558 upper=0.43633231299858238339 effort=0.52 velocity=10.7
- joint right_hip_yaw: limit lower=-0.69813170079773179122 upper=0.69813170079773179122 effort=1.0 velocity=10.7 -> lower=-0.69813170079773179122 upper=0.69813170079773179122 effort=0.52 velocity=10.7
- joint right_knee: limit lower=-2.0943951023931952626 upper=2.0943951023931952626 effort=1.0 velocity=10.7 -> lower=-2.0943951023931952626 upper=2.0943951023931952626 effort=0.52 velocity=10.7

Commit message: 1 nm knee efort

File: assets/urdf/bdx/urdf/bdx.urdf (robot description, URDF)
Before this commit: robot bdx, 20 links, 19 joints
Joints:
- joint left_knee: limit lower=-2.0943951023931952626 upper=2.0943951023931952626 effort=0.52 velocity=10.7 -> lower=-2.0943951023931952626 upper=2.0943951023931952626 effort=0.9 velocity=10.7
- joint right_knee: limit lower=-2.0943951023931952626 upper=2.0943951023931952626 effort=0.52 velocity=10.7 -> lower=-2.0943951023931952626 upper=2.0943951023931952626 effort=0.9 velocity=10.7
